Commit message: adjust urdf

File: urdf/drone.urdf (robot description, URDF)
Before this commit: robot drone, 5 links, 4 joints
Joints:
- joint lidar_joint: origin xyz=0 0 -0.075 rpy=0 0 0 -> xyz=0 0 -0.075 rpy=0 0 3.14159

Commit message: adjust param

File: urdf/drone.urdf (robot description, URDF)
Before this commit: robot drone, 5 links, 4 joints
Joints:
- joint camera_joint: origin xyz=0.145 0 0.0 rpy=0 0 0 -> xyz=0.17 0 0.0 rpy=0 0 0
- joint imu_joint: origin xyz=0.0 0.0 0.02 rpy=0 0 0 -> xyz=0.0 0.0 0.0 rpy=0 0 0
- joint lidar_joint: origin xyz=0 0 -0.075 rpy=0 0 3.14159 -> xyz=0 0 0.11 rpy=0 0 3.14159
